Commit message: added new file

File: myrobot/urdf/myrobot.urdf.xacro (robot description, xacro)
@@ -57,5 +57,5 @@
     <visual>
       <geometry>
-        <box size="${base_len} ${base_width} 0.02"/>
+        <box size="${base_len} ${base_width} 0.05"/>
       </geometry>
       <material name="black"/>
@@ -63,5 +63,5 @@
     <collision>
       <geometry>
-        <box size="${base_len} ${base_width} 0.01"/>
+        <box size="${base_len} ${base_width} 0.05"/>
       </geometry>
     </collision>

Commit message: added fingers

File: myrobot/urdf/myrobot.urdf.xacro (robot description, xacro)
@@ -48,5 +48,5 @@
         <origin xyz="0 0 0" rpy="0 0 0" />
         <geometry>
-            <box size="0.001 0.001 0.001" />
+            <box size="0.001 0.001 0.05" />
         </geometry>
     </visual>
@@ -57,5 +57,5 @@
     <visual>
       <geometry>
-        <box size="${base_len} ${base_width} 0.05"/>
+        <box size="${base_len} ${base_width} 0.1"/>
       </geometry>
       <material name="black"/>
@@ -63,5 +63,5 @@
     <collision>
       <geometry>
-        <box size="${base_len} ${base_width} 0.05"/>
+        <box size="${base_len} ${base_width} 0.1"/>
       </geometry>
     </collision>
@@ -108,5 +108,5 @@
         <sphere radius="${caster_wheel_radius}"/>
       </geometry>
-      <material name="blue"/>
+      <material name="black"/>
     </visual>
     <collision>
@@ -125,4 +125,86 @@
     <origin xyz="${caster_wheel_joint_offset} 0 -${caster_wheel_radius+0.005}" rpy="0 0 0"/>
   </joint>
+<!--left guide-->
+<link name="left_guide">
+  <xacro:box_inertia m="1" w="${base_len}" h="${base_width}" d="0.01"/>
+  <visual>
+    <geometry>
+      <box size="0.5 0.01 0.05"/>
+    </geometry>
+  <link name="left_guide">
+    <xacro:box_inertia m="1" w="${base_len}" h="${base_width}" d="0.01"/>
+    <visual>
+      <geometry>
+        <box size="0.5 0.01 0.05"/>
+      </geometry>
+      <material name="blue"/>
+    </visual>
+    <collision>
+      <geometry>
+        <box size="0.5 0.01 0.05"/>
+      </geometry>
+    </collision>
+  </link>
+  <!--left_guide to left_guide Joint-->
+  <joint name="left_guide_joint" type="fixed">
+    <origin xyz="-0.2 0.5 0.0" rpy="0 0 0" />
+    <parent link="base_footprint"/>
+    <child link="left_guide" />
+  </joint>
+    <material name="blue"/>
+  </visual>
+  <collision>
+    <geometry>
+      <box size="0.5 0.01 0.05"/>
+    </geometry>
+  </collision>
+</link>
+<!--left_guide to left_guide Joint-->
+<joint name="left_guide_joint" type="fixed">
+  <origin xyz="-0.2 0.15 0.06" rpy="0 0 0" />
+  <parent link="base_footprint"/>
+  <child link="left_guide" />
+</joint>
+<!--right guide-->
+<link name="right_guide">
+  <xacro:box_inertia m="1" w="${base_len}" h="${base_width}" d="0.01"/>
+  <visual>
+    <geometry>
+      <box size="0.5 0.01 0.05"/>
+    </geometry>
+  <link name="right_guide">
+    <xacro:box_inertia m="1" w="${base_len}" h="${base_width}" d="0.01"/>
+    <visual>
+      <geometry>
+        <box size="0.5 0.01 0.05"/>
+      </geometry>
+      <material name="blue"/>
+    </visual>
+    <collision>
+      <geometry>
+        <box size="0.5 0.01 0.05"/>
+      </geometry>
+    </collision>
+  </link>
+  <!--right_guide to right_guide Joint-->
+  <joint name="right_guide_joint" type="fixed">
+    <origin xyz="-0.2 0.5 0.0" rpy="0 0 0" />
+    <parent link="base_footprint"/>
+    <child link="right_guide" />
+  </joint>
+    <material name="blue"/>
+  </visual>
+  <collision>
+    <geometry>
+      <box size="0.5 0.01 0.05"/>
+    </geometry>
+  </collision>
+</link>
+<!--right_guide to right_guide Joint-->
+<joint name="right_guide_joint" type="fixed">
+  <origin xyz="-0.2 -0.15 0.06" rpy="0 0 0" />
+  <parent link="base_footprint"/>
+  <child link="right_guide" />
+</joint>
   <xacro:include filename="$(find myrobot)/urdf/myrobot_pluggin.xacro"/>
 </robot>

Commit message: added support

File: myrobot/urdf/myrobot.urdf.xacro (robot description, xacro)
@@ -207,4 +207,45 @@
   <child link="right_guide" />
 </joint>
+<!--body guide-->
+<link name="body_guide">
+  <xacro:box_inertia m="1" w="${base_len}" h="${base_width}" d="0.01"/>
+  <visual>
+    <geometry>
+      <box size="0.2 0.2 0.3"/>
+    </geometry>
+  <link name="body_guide">
+    <xacro:box_inertia m="1" w="${base_len}" h="${base_width}" d="0.01"/>
+    <visual>
+      <geometry>
+        <box size="0.2 0.2 0.3"/>
+      </geometry>
+      <material name="blue"/>
+    </visual>
+    <collision>
+      <geometry>
+        <box size="0.2 0.2 0.3"/>
+      </geometry>
+    </collision>
+  </link>
+  <!--body_guide to body_guide Joint-->
+  <joint name="body_guide_joint" type="fixed">
+    <origin xyz="0 0 1" rpy="0 0 0" />
+    <parent link="base_footprint"/>
+    <child link="body_guide" />
+  </joint>
+    <material name="blue"/>
+  </visual>
+  <collision>
+    <geometry>
+      <box size="0.2 0.2 0.3"/>
+    </geometry>
+  </collision>
+</link>0
+<!--body_guide to body_guide Joint-->
+<joint name="body_guide_joint" type="fixed">
+  <origin xyz="0 0 0.2" rpy="0 0 0" />
+  <parent link="base_footprint"/>
+  <child link="body_guide" />
+</joint>
   <xacro:include filename="$(find myrobot)/urdf/myrobot_pluggin.xacro"/>
 </robot>

Commit message: changed colors

File: myrobot/urdf/myrobot.urdf.xacro (robot description, xacro)
@@ -108,5 +108,5 @@
         <sphere radius="${caster_wheel_radius}"/>
       </geometry>
-      <material name="black"/>
+      <material name="red"/>
     </visual>
     <collision>
@@ -220,5 +220,5 @@
         <box size="0.2 0.2 0.3"/>
       </geometry>
-      <material name="blue"/>
+      <material name="red"/>
     </visual>
     <collision>
@@ -234,5 +234,5 @@
     <child link="body_guide" />
   </joint>
-    <material name="blue"/>
+    <material name="red"/>
   </visual>
   <collision>
